File: KiCAD/Arduino 7segment timer.kicad_pcb (KiCad board)
At the start: 2 copper layers, 7.1 x 10.2 mm, 43 parts, among them J1 AC, J2 DC 12V, J3 LOAD, J5 HEADER_3, J6 HEADER_3, Q1 BC847, Q2 BC847, Q3 BC847, Q4 BC847, Q5 BC847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

Commit message: PCB updated
to include CC and OSH logos
Parts:
- added REF**: Symbol_CC-Noncommercial_CopperTop_Small, Symbols:Symbol_CC-Noncommercial_CopperTop_Small, F.Cu at (47.0, 106.2)
- added REF**: Symbol_CreativeCommons_CopperTop_Type2_Small, Symbols:Symbol_CreativeCommons_CopperTop_Type2_Small, F.Cu at (90.7, 50.8)
- added REF**: Symbol_OSHW-Logo_SilkScreen, Symbols:Symbol_OSHW-Logo_SilkScreen, F.Cu at (90.7, 42.7)
- added REF**: Symbol_OSHW-Logo_CopperTop, Symbols:Symbol_OSHW-Logo_CopperTop, F.Cu at (90.7, 42.7)
- moved R11 5.80 mm to (45.7, 87.6)
- moved SP1 2.03 mm to (46.5, 94.0)
Routing:
- net /Control/Buzzer: track 45.1 -> 47.4 mm
- net Net-(Q5-Pad3): track 7.54 -> 5.43 mm
- net Net-(R10-Pad2): track 4.46 -> 6.49 mm
Other:
- board text added: "CDTimer 4 Ard"
- board text added: "ejs 2016"
